File: placaCub/placaCub.kicad_pcb (KiCad board)
At the start: 2 copper layers, 112 parts, among them J1 conector UART, J10 conector fila 6, J11 conector fila 7, J12 conector columna 0, J13 conector columna 1, J14 conector columna 2, J15 conector columna 3, J16 conector columna 4, J17 conector columna 5, J18 conector columna 6, J19 conector columna 7, J2 conector I2C, J20 conector botones, J21 Conn_01x05_Male, J3 conector energia, J4 coenctor fila 0, J5 conector fila 1, J6 conector fila 2, J7 conector fila 3, J8 conector fila 4, J9 conector fila 5, Q1 BD241C, Q2 BD241C, Q3 BD241C, Q4 BD241C, Q5 BD241C, Q6 BD241C, Q7 BD241C, Q8 BD241C, SW1 SW_MEC_5E, SW2 SW_MEC_5E, SW3 SW_MEC_5E, SW4 SW_MEC_5E, U1 YAAJ_BluePill_Part_Like, U10 74AHC595, U2 74AHC595, U3 74AHC595, U4 74AHC595, U5 74AHC595, U6 74AHC595, U7 74AHC595, U8 74AHC595, U9 74AHC595

Commit message: diseño del pcb
Parts:
- moved J16 261.4 mm to (118.9, 278.9), turned to 90 degrees
- moved U10 246.5 mm to (94.5, 153.9), turned to 180 degrees
- moved J18 238.0 mm to (118.9, 213.4), turned to 90 degrees
- moved J17 230.9 mm to (119.4, 247.4), turned to 90 degrees
- moved R60 230.0 mm to (110.5, 268.7), turned to 180 degrees
- moved R27 227.4 mm to (110.5, 275.8), turned to 180 degrees
- moved R44 221.3 mm to (110.5, 265.2), turned to 180 degrees
- moved R30 197.8 mm to (110.2, 228.1), turned to 180 degrees
- moved U9 192.7 mm to (94.5, 180.3), turned to 180 degrees
- moved R62 176.7 mm to (110.2, 235.2), turned to 180 degrees
- moved R43 176.2 mm to (110.5, 279.4), turned to 180 degrees
- moved R45 175.4 mm to (110.2, 245.9), turned to 180 degrees
- moved R47 168.5 mm to (110.2, 213.9), turned to 180 degrees
- moved R12 167.3 mm to (110.5, 258.1), turned to 180 degrees
- moved R31 165.3 mm to (110.2, 210.3), turned to 180 degrees
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
Commit message: avances en el diseño del PCB
Parts:
- moved U10 99.5 mm to (124.0, 58.9)
- moved U2 98.8 mm to (72.1, 72.6)
- moved R19 98.7 mm to (55.9, 76.2)
- moved R3 98.6 mm to (55.9, 79.8)
- moved R12 98.4 mm to (123.4, 160.5)
- moved R59 98.4 mm to (123.4, 185.4)
- moved R60 98.4 mm to (123.4, 171.2)
- moved R11 98.4 mm to (123.4, 174.8)
- moved R27 98.4 mm to (123.4, 178.3)
- moved R28 98.4 mm to (123.4, 164.1)
- moved R44 98.4 mm to (123.4, 167.6)
- moved R43 98.4 mm to (123.4, 181.9)
- moved R52 98.4 mm to (55.9, 83.3)
- moved R35 98.3 mm to (55.9, 72.6)
- moved R51 98.3 mm to (55.9, 69.1)
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Routing:
- net MOSI: track 0.00 -> 22.1 mm
- net Net-(U2-Pad9): track 0.00 -> 20.3 mm
- net Net-(U3-Pad9): track 0.00 -> 20.2 mm
- net Net-(R65-Pad2): track 0.00 -> 16.2 mm
- net Net-(R61-Pad2): track 0.00 -> 16.2 mm
- net Net-(R63-Pad2): track 0.00 -> 16.2 mm
- net Net-(R57-Pad2): track 0.00 -> 16.2 mm
- net Net-(R55-Pad2): track 0.00 -> 16.2 mm
- net Net-(R53-Pad2): track 0.00 -> 16.2 mm
- net Net-(R51-Pad2): track 0.00 -> 16.2 mm
- net Net-(R59-Pad2): track 0.00 -> 16.2 mm
- net TX: track 0.00 -> 15.8 mm
- net RX: track 0.00 -> 15.8 mm
- net SDA: track 0.00 -> 15.0 mm
- net SCL: track 0.00 -> 15.0 mm
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Other:
- net class Default: clearance 0.2 -> 1.15; trace_width 0.25 -> 0.7; via_dia 0.8 -> 2; via_drill 0.4 -> 1
- rule trace_clearance: 0.2 -> 1.15

Commit message: nuevo update 28/03/2022
Routing:
- net +5V: track 0.00 -> 541.5 mm
- net SCK: track 1.20 -> 221.5 mm, vias 0 -> 2
- net STORE: track 0.00 -> 201.4 mm, vias 0 -> 14
- net Net-(U5-Pad9): track 0.00 -> 25.8 mm
- net Net-(U4-Pad9): track 0.00 -> 20.3 mm
- net Net-(U8-Pad9): track 0.00 -> 20.3 mm
- net Net-(U7-Pad9): track 0.00 -> 20.2 mm
- net Net-(U6-Pad9): track 1.13 -> 20.3 mm
- net Net-(R61-Pad2): track 16.2 -> 18.2 mm
- net Net-(R63-Pad2): track 16.2 -> 18.0 mm
- net Net-(R65-Pad2): track 16.2 -> 18.0 mm

Commit message: contornos de la placa realizados
Parts:
- moved J3 111.4 mm to (45.2, 55.9), turned to 270 degrees
- moved D1 110.7 mm to (48.8, 34.5), turned to 180 degrees
- moved D2 110.2 mm to (48.8, 40.1), turned to 180 degrees
- moved C1 97.5 mm to (56.4, 62.0), turned to 90 degrees
- moved R2 97.1 mm to (55.9, 42.7), turned to 270 degrees
- moved R1 93.1 mm to (60.5, 38.6), turned to 270 degrees
- moved Q8 60.6 mm to (153.9, 34.0), turned to 270 degrees
- moved J11 57.8 mm to (165.1, 36.6)
- moved Q7 56.1 mm to (153.9, 51.3), turned to 270 degrees
- moved J10 53.2 mm to (165.1, 53.8)
- moved Q6 48.1 mm to (153.9, 71.6), turned to 270 degrees
- moved J9 45.2 mm to (165.1, 74.2)
- moved Q5 39.2 mm to (153.9, 92.5), turned to 270 degrees
- moved J8 36.2 mm to (165.1, 95.0)
- moved Q4 28.4 mm to (153.9, 115.3), turned to 270 degrees
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Routing:
- net +5V: track 541.5 -> 677.4 mm
- net Net-(Q1-Pad1): track 0.00 -> 133.5 mm
- net Net-(Q2-Pad1): track 0.00 -> 108.8 mm
- net Net-(Q3-Pad1): track 0.00 -> 87.0 mm
- net Net-(Q4-Pad1): track 0.00 -> 69.3 mm
- net Net-(Q5-Pad1): track 0.00 -> 49.0 mm
- net SCK: track 221.5 -> 264.3 mm
- net STORE: track 201.4 -> 241.9 mm
- net Net-(U10-Pad14): track 0.00 -> 39.8 mm
- net Net-(Q6-Pad1): track 0.00 -> 30.8 mm
- net Net-(R1-Pad2): track 0.00 -> 28.9 mm, vias 0 -> 2
- net Net-(R2-Pad2): track 0.00 -> 27.4 mm, vias 0 -> 2
- net Net-(Q8-Pad1): track 0.00 -> 22.4 mm
- net Net-(Q7-Pad1): track 0.00 -> 18.4 mm
- net Net-(D1-Pad1): track 0.00 -> 13.4 mm
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Other:
- board outline added: 132.6 x 169.7 mm

Commit message: archivo CNC en proceso
Parts:
- SW1: value SW_MEC_5E -> boton arriba
- SW2: value SW_MEC_5E -> boton abajo
- SW3: value SW_MEC_5E -> boton izquierda
- SW4: value SW_MEC_5E -> boton derecha
- moved SW4 58.2 mm to (248.5, 45.7)
- moved SW1 53.4 mm to (238.4, 34.6)
- moved SW3 48.0 mm to (228.1, 45.7)
- moved SW2 45.2 mm to (238.4, 56.9)
- moved J21 34.1 mm to (223.5, 68.6)
- moved J4 6.10 mm to (165.1, 174.8)
- moved J5 6.10 mm to (165.1, 156.5)
- moved Q1 6.10 mm to (153.9, 172.2)
- moved Q2 6.10 mm to (153.9, 153.9)
- moved J10 4.57 mm to (165.1, 58.4)
- moved Q7 4.57 mm to (153.9, 55.9)
- moved J11 3.05 mm to (165.1, 39.6)
- moved Q6 3.05 mm to (153.9, 74.7)
- moved Q8 3.05 mm to (153.9, 37.1)
- moved J9 3.05 mm to (165.1, 77.2)
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Routing:
- net 0: track 0.00 -> 84.8 mm, vias 0 -> 20
- net +5V: track 677.4 -> 749.4 mm, vias 0 -> 2
- net Net-(Q2-Pad1): track 108.8 -> 101.7 mm
- net Net-(Q1-Pad1): track 133.5 -> 126.4 mm
- net Net-(Q6-Pad1): track 30.8 -> 33.8 mm
- net Net-(Q7-Pad1): track 18.4 -> 21.0 mm
- net Net-(Q3-Pad1): track 87.0 -> 84.5 mm
- net Net-(Q8-Pad1): track 22.4 -> 20.0 mm
- net Net-(Q4-Pad1): track 69.3 -> 67.2 mm
- net Net-(D1-Pad1): track 13.4 -> 12.3 mm
- net Net-(D2-Pad1): track 8.16 -> 7.11 mm
- net Net-(Q5-Pad1): track 49.0 -> 50.0 mm
- added copper zone on B.Cu, net (none)
- added copper zone on B.Cu, net 0
Other:
- outline, holes or cut-outs redrawn
