File: placaCub/placaCub.sch (KiCad schematic (older format))
At the start: 112 parts, among them J1 conector UART, J10 conector fila 6, J11 conector fila 7, J12 conector columna 0, J13 conector columna 1, J14 conector columna 2, J15 conector columna 3, J16 conector columna 4, J17 conector columna 5, J18 conector columna 6, J19 conector columna 7, J2 conector I2C, J20 conector botones, J21 Conn_01x05_Male, J3 conector energia, J4 coenctor fila 0, J5 conector fila 1, J6 conector fila 2, J7 conector fila 3, J8 conector fila 4, J9 conector fila 5, Q1 BD241C, Q2 BD241C, Q3 BD241C, Q4 BD241C, Q5 BD241C, Q6 BD241C, Q7 BD241C, Q8 BD241C, SW1 SW_MEC_5E, SW2 SW_MEC_5E, SW3 SW_MEC_5E, SW4 SW_MEC_5E, U1 YAAJ_BluePill_Part_Like, U10 74AHC595, U2 74AHC595, U3 74AHC595, U4 74AHC595, U5 74AHC595, U6 74AHC595, U7 74AHC595, U8 74AHC595, U9 74AHC595

Commit message: diseño del pcb
Parts:
- U1: symbol STM32_BluePill:YAAJ_BluePill_Part_Like -> placaCub-rescue:YAAJ_BluePill_Part_Like-STM32_BluePill
Changed lines of the file:
@@
 $EndComp
 $Comp
-L STM32_BluePill:YAAJ_BluePill_Part_Like U1
+L placaCub-rescue:YAAJ_BluePill_Part_Like-STM32_BluePill U1
 U 1 1 623AC22C
 P 5750 4000

Commit message: archivo CNC en proceso
Parts:
- SW1: value SW_MEC_5E -> boton arriba
- SW2: value SW_MEC_5E -> boton abajo
- SW3: value SW_MEC_5E -> boton izquierda
- SW4: value SW_MEC_5E -> boton derecha
Changed lines of the file:
@@
 P 7850 1400
 F 0 "SW1" H 7850 1785 50  0000 C CNN
-F 1 "SW_MEC_5E" H 7850 1694 50  0000 C CNN
+F 1 "boton arriba" H 7850 1694 50  0000 C CNN
 F 2 "Button_Switch_THT:SW_PUSH_6mm_H7.3mm" H 7850 1700 50  0001 C CNN
 F 3 "http://www.apem.com/int/index.php?controller=attachment&id_attachment=1371" H 7850 1700 50  0001 C CNN
@@
 P 7850 2400
 F 0 "SW3" H 7850 2785 50  0000 C CNN
-F 1 "SW_MEC_5E" H 7850 2694 50  0000 C CNN
+F 1 "boton izquierda" H 7850 2694 50  0000 C CNN
 F 2 "Button_Switch_THT:SW_PUSH_6mm_H7.3mm" H 7850 2700 50  0001 C CNN
 F 3 "http://www.apem.com/int/index.php?controller=attachment&id_attachment=1371" H 7850 2700 50  0001 C CNN
@@
 P 7850 1900
 F 0 "SW2" H 7850 2285 50  0000 C CNN
-F 1 "SW_MEC_5E" H 7850 2194 50  0000 C CNN
+F 1 "boton abajo" H 7850 2194 50  0000 C CNN
 F 2 "Button_Switch_THT:SW_PUSH_6mm_H7.3mm" H 7850 2200 50  0001 C CNN
 F 3 "http://www.apem.com/int/index.php?controller=attachment&id_attachment=1371" H 7850 2200 50  0001 C CNN
@@
 P 7850 2900
 F 0 "SW4" H 7850 3285 50  0000 C CNN
-F 1 "SW_MEC_5E" H 7850 3194 50  0000 C CNN
+F 1 "boton derecha" H 7850 3194 50  0000 C CNN
 F 2 "Button_Switch_THT:SW_PUSH_6mm_H7.3mm" H 7850 3200 50  0001 C CNN
 F 3 "http://www.apem.com/int/index.php?controller=attachment&id_attachment=1371" H 7850 3200 50  0001 C CNN
